File: main.kicad_pcb (KiCad board)
At the start: 2 copper layers, 4 parts, among them M1 XBEE, U1 BME280, U2 NCS36000

Commit message: test
Parts:
- M1: footprint BME280:XBEE -> XBEE:XBEE-SMD
Changed lines of the file:
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@@
     (links 5)
     (no_connects 5)
-    (area 176.317299 87.211559 201.577248 117.47688)
+    (area 174.165194 85.846309 202.57704 120.658231)
     (thickness 1.6)
     (drawings 0)
@@
     )
   )
-  (module BME280:XBEE (layer F.Cu)
+  (module XBEE:XBEE-SMD (layer F.Cu)
     (at 188.7982 104.22128)
-    (attr virtual)
-    (fp_text reference M1 (at -10.414 12.192) (layer F.SilkS)
+    (attr smd)
+    (fp_text reference M1 (at 0 8.99922) (layer F.SilkS)
       (effects (font (size 1.016 1.016) (thickness 0.1016)))
     )
-    (fp_text value XBEE (at 10.668 12.192) (layer F.SilkS)
-      (effects (font (size 1.016 1.016) (thickness 0.1016)))
-    )
-    (fp_line (start -12.192 10.88644) (end 12.192 10.88644) (layer F.SilkS) (width 0.1778))
-    (fp_line (start 12.192 10.88644) (end 12.192 -9.398) (layer F.SilkS) (width 0.1778))
-    (fp_line (start 12.192 -9.398) (end 4.86664 -16.72082) (layer F.SilkS) (width 0.1778))
-    (fp_line (start 4.86664 -16.72082) (end -4.86664 -16.72082) (layer F.SilkS) (width 0.1778))
-    (fp_line (start -4.86664 -16.72082) (end -12.192 -9.398) (layer F.SilkS) (width 0.1778))
-    (fp_line (start -12.192 -9.398) (end -12.192 10.88644) (layer F.SilkS) (width 0.1778))
-    (fp_line (start -12.192 10.88644) (end 12.192 10.88644) (layer F.SilkS) (width 0.127))
-    (fp_line (start 12.192 10.88644) (end 12.192 -9.398) (layer F.SilkS) (width 0.127))
-    (fp_line (start 12.192 -9.398) (end 4.86664 -16.72082) (layer F.SilkS) (width 0.127))
-    (fp_line (start 4.86664 -16.72082) (end -4.86664 -16.72082) (layer F.SilkS) (width 0.127))
-    (fp_line (start -4.86664 -16.72082) (end -12.192 -9.398) (layer F.SilkS) (width 0.127))
-    (fp_line (start -12.192 -9.398) (end -12.192 10.88644) (layer F.SilkS) (width 0.127))
-    (pad 1 thru_hole circle (at -10.9982 -8.99922) (size 1.1684 1.1684) (drill 0.6604) (layers *.Cu *.Mask F.Paste F.SilkS)
+    (fp_text value XBEE (at -12.99972 -11.00074) (layer F.SilkS)
+      (effects (font (size 0.762 0.762) (thickness 0.1016)))
+    )
+    (fp_line (start 12.30122 -13.12418) (end 4.95046 -18.12544) (layer F.SilkS) (width 0.09906))
+    (fp_line (start -12.10056 -13.12418) (end -4.7752 -18.12544) (layer F.SilkS) (width 0.09906))
+    (fp_line (start -12.192 16.18742) (end 12.192 16.18742) (layer F.SilkS) (width 0.09906))
+    (fp_line (start 4.94284 -18.12036) (end -4.79044 -18.12036) (layer F.SilkS) (width 0.09906))
+    (pad 2 smd rect (at -13.0048 -7.00024 270) (size 0.889 2.29108) (layers F.Cu F.Paste F.Mask)
+      (net 22 "Net-(M1-Pad2)"))
+    (pad 4 smd rect (at -13.0048 -2.99974 270) (size 0.889 2.29108) (layers F.Cu F.Paste F.Mask)
+      (net 24 "Net-(M1-Pad4)"))
+    (pad 6 smd rect (at -13.0048 1.00076 270) (size 0.889 2.29108) (layers F.Cu F.Paste F.Mask)
+      (net 26 "Net-(M1-Pad6)"))
+    (pad 8 smd rect (at -13.0048 5.00126 270) (size 0.889 2.29108) (layers F.Cu F.Paste F.Mask)
+      (net 28 "Net-(M1-Pad8)"))
+    (pad 10 smd rect (at -13.0048 9.00176 270) (size 0.889 2.29108) (layers F.Cu F.Paste F.Mask)
+      (net 1 GND))
+    (pad 9 smd rect (at -9.0678 7.00024 270) (size 0.889 2.29108) (layers F.Cu F.Paste F.Mask)
+      (net 29 "Net-(M1-Pad9)"))
+    (pad 7 smd rect (at -9.0678 2.99974 270) (size 0.889 2.29108) (layers F.Cu F.Paste F.Mask)
+      (net 27 "Net-(M1-Pad7)"))
+    (pad 5 smd rect (at -9.0678 -1.00076 270) (size 0.889 2.29108) (layers F.Cu F.Paste F.Mask)
+      (net 25 "Net-(M1-Pad5)"))
+    (pad 3 smd rect (at -9.0678 -4.99872 270) (size 0.889 2.29108) (layers F.Cu F.Paste F.Mask)
+      (net 23 "Net-(M1-Pad3)"))
+    (pad 1 smd rect (at -9.0678 -8.99922 270) (size 0.889 2.29108) (layers F.Cu F.Paste F.Mask)
       (net 6 +3V3))
-    (pad 2 thru_hole circle (at -10.9982 -6.9977) (size 1.1684 1.1684) (drill 0.6604) (layers *.Cu *.Mask F.Paste F.SilkS)
-      (net 22 "Net-(M1-Pad2)"))
-    (pad 3 thru_hole circle (at -10.9982 -4.99872) (size 1.1684 1.1684) (drill 0.6604) (layers *.Cu *.Mask F.Paste F.SilkS)
-      (net 23 "Net-(M1-Pad3)"))
-    (pad 4 thru_hole circle (at -10.9982 -2.99974) (size 1.1684 1.1684) (drill 0.6604) (layers *.Cu *.Mask F.Paste F.SilkS)
-      (net 24 "Net-(M1-Pad4)"))
-    (pad 5 thru_hole circle (at -10.9982 -0.99822) (size 1.1684 1.1684) (drill 0.6604) (layers *.Cu *.Mask F.Paste F.SilkS)
-      (net 25 "Net-(M1-Pad5)"))
-    (pad 6 thru_hole circle (at -10.9982 0.99822) (size 1.1684 1.1684) (drill 0.6604) (layers *.Cu *.Mask F.Paste F.SilkS)
-      (net 26 "Net-(M1-Pad6)"))
-    (pad 7 thru_hole circle (at -10.9982 2.99974) (size 1.1684 1.1684) (drill 0.6604) (layers *.Cu *.Mask F.Paste F.SilkS)
-      (net 27 "Net-(M1-Pad7)"))
-    (pad 8 thru_hole circle (at -10.9982 4.99872) (size 1.1684 1.1684) (drill 0.6604) (layers *.Cu *.Mask F.Paste F.SilkS)
-      (net 28 "Net-(M1-Pad8)"))
-    (pad 9 thru_hole circle (at -10.9982 6.9977) (size 1.1684 1.1684) (drill 0.6604) (layers *.Cu *.Mask F.Paste F.SilkS)
-      (net 29 "Net-(M1-Pad9)"))
-    (pad 10 thru_hole circle (at -10.9982 8.99922) (size 1.1684 1.1684) (drill 0.6604) (layers *.Cu *.Mask F.Paste F.SilkS)
-      (net 1 GND))
-    (pad 11 thru_hole circle (at 10.9982 8.99922) (size 1.1684 1.1684) (drill 0.6604) (layers *.Cu *.Mask F.Paste F.SilkS)
+    (pad 20 smd rect (at 12.4333 -8.99922 270) (size 0.889 2.29108) (layers F.Cu F.Paste F.Mask)
+      (net 39 "Net-(M1-Pad20)"))
+    (pad 19 smd rect (at 8.49884 -7.00024 270) (size 0.889 2.29108) (layers F.Cu F.Paste F.Mask)
+      (net 38 "Net-(M1-Pad19)"))
+    (pad 18 smd rect (at 12.4333 -4.99872 270) (size 0.889 2.29108) (layers F.Cu F.Paste F.Mask)
+      (net 37 "Net-(M1-Pad18)"))
+    (pad 17 smd rect (at 8.49884 -2.99974 270) (size 0.889 2.29108) (layers F.Cu F.Paste F.Mask)
+      (net 36 "Net-(M1-Pad17)"))
+    (pad 16 smd rect (at 12.4333 -1.00076 270) (size 0.889 2.29108) (layers F.Cu F.Paste F.Mask)
+      (net 35 "Net-(M1-Pad16)"))
+    (pad 15 smd rect (at 8.49884 1.00076 270) (size 0.889 2.29108) (layers F.Cu F.Paste F.Mask)
+      (net 34 "Net-(M1-Pad15)"))
+    (pad 14 smd rect (at 12.4333 2.99974 270) (size 0.889 2.29108) (layers F.Cu F.Paste F.Mask)
+      (net 33 "Net-(M1-Pad14)"))
+    (pad 13 smd rect (at 8.49884 5.00126 270) (size 0.889 2.29108) (layers F.Cu F.Paste F.Mask)
+      (net 32 "Net-(M1-Pad13)"))
+    (pad 12 smd rect (at 12.4333 7.00024 270) (size 0.889 2.29108) (layers F.Cu F.Paste F.Mask)
+      (net 31 "Net-(M1-Pad12)"))
+    (pad 11 smd rect (at 8.4328 9.00176 270) (size 0.889 2.29108) (layers F.Cu F.Paste F.Mask)
       (net 30 "Net-(M1-Pad11)"))
-    (pad 12 thru_hole circle (at 10.9982 6.9977) (size 1.1684 1.1684) (drill 0.6604) (layers *.Cu *.Mask F.Paste F.SilkS)
-      (net 31 "Net-(M1-Pad12)"))
-    (pad 13 thru_hole circle (at 10.9982 4.99872) (size 1.1684 1.1684) (drill 0.6604) (layers *.Cu *.Mask F.Paste F.SilkS)
-      (net 32 "Net-(M1-Pad13)"))
-    (pad 14 thru_hole circle (at 10.9982 2.99974) (size 1.1684 1.1684) (drill 0.6604) (layers *.Cu *.Mask F.Paste F.SilkS)
-      (net 33 "Net-(M1-Pad14)"))
-    (pad 15 thru_hole circle (at 10.9982 0.99822) (size 1.1684 1.1684) (drill 0.6604) (layers *.Cu *.Mask F.Paste F.SilkS)
-      (net 34 "Net-(M1-Pad15)"))
-    (pad 16 thru_hole circle (at 10.9982 -0.99822) (size 1.1684 1.1684) (drill 0.6604) (layers *.Cu *.Mask F.Paste F.SilkS)
-      (net 35 "Net-(M1-Pad16)"))
-    (pad 17 thru_hole circle (at 10.9982 -2.99974) (size 1.1684 1.1684) (drill 0.6604) (layers *.Cu *.Mask F.Paste F.SilkS)
-      (net 36 "Net-(M1-Pad17)"))
-    (pad 18 thru_hole circle (at 10.9982 -4.99872) (size 1.1684 1.1684) (drill 0.6604) (layers *.Cu *.Mask F.Paste F.SilkS)
-      (net 37 "Net-(M1-Pad18)"))
-    (pad 19 thru_hole circle (at 10.9982 -6.9977) (size 1.1684 1.1684) (drill 0.6604) (layers *.Cu *.Mask F.Paste F.SilkS)
-      (net 38 "Net-(M1-Pad19)"))
-    (pad 20 thru_hole circle (at 10.9982 -8.99922) (size 1.1684 1.1684) (drill 0.6604) (layers *.Cu *.Mask F.Paste F.SilkS)
-      (net 39 "Net-(M1-Pad20)"))
   )
 )

Commit message: test
Parts:
- added C2: 10µF, Capacitors_SMD:CP_Elec_3x5.3, F.Cu at (241.3, 94.0)
- added C3: 0.1µF, Capacitors_SMD:C_0402, F.Cu at (242.4, 86.1)
- added C4: 0.1µF, Capacitors_SMD:C_0402, F.Cu at (235.5, 119.4)
- added R1: 4.7k, Resistors_SMD:R_0402, F.Cu at (228.3, 94.0)
- added R2: 4.7k, Resistors_SMD:R_0402, F.Cu at (246.8, 126.9)
- added R3: 0, Resistors_SMD:R_0402, F.Cu at (231.3, 94.0)
- added R4: 0, Resistors_SMD:R_0402, F.Cu at (227.7, 98.8)
- added SW1: Reset, Buttons_Switches_SMD:SW_SPST_B3S-1000, F.Cu at (227.3, 132.1)
- C1: value CP -> 10µF
- M1: value XBEE -> mDot; footprint XBEE:XBEE-SMD -> XBEE:XBEE
- moved U1 57.7 mm to (237.8, 88.2)
- moved M1 44.7 mm to (232.2, 114.8)
- moved C1 44.6 mm to (229.3, 87.7)
- moved U2 41.6 mm to (229.9, 109.2)
Connections:
- U1 pad 2: Net-(U1-Pad2) -> +3V3
- U1 pad 3: Net-(U1-Pad3) -> Net-(M1-Pad7)
- U1 pad 4: Net-(U1-Pad4) -> Net-(M1-Pad6)
- U1 pad 6: Net-(U1-Pad6) -> +3V3
- U1 pad 7: Net-(U1-Pad7) -> GND

Commit message: test
Parts:
- removed R3, R4: 0, Resistors_SMD:R_0402
- added C10: 100nF, Capacitors_SMD:C_0402, F.Cu at (245.9, 79.2)
- added C5: 33µF, Capacitors_SMD:C_0805, F.Cu at (249.4, 92.7)
- added C6: 33µF, Capacitors_SMD:C_0805, F.Cu at (247.7, 92.7)
- added C7: 100nF, Capacitors_SMD:C_0402, F.Cu at (249.7, 89.7)
- added C8: 10nF, Capacitors_SMD:C_0402, F.Cu at (245.8, 88.9)
- added C9: 100nF, Capacitors_SMD:C_0402, F.Cu at (251.7, 89.7)
- added R5: 10k, Resistors_SMD:R_0402, F.Cu at (251.0, 92.7)
- added R6: 10k, Resistors_SMD:R_0402, F.Cu at (248.2, 88.9)
- added R7: 10k, Resistors_SMD:R_0402, F.Cu at (246.4, 90.2)
- added R8: 43k, Resistors_SMD:R_0402, F.Cu at (250.7, 89.6)
- added R9: 51k, Resistors_SMD:R_0402, F.Cu at (246.9, 79.2)
- added RV1: 1M, Potentiometers:Potentiometer_Trimmer-EVM3E, F.Cu at (241.3, 89.7)
- added RV2: 1M, Potentiometers:Potentiometer_Trimmer-EVM3E, F.Cu at (241.8, 75.7)
- added U3: NCS36000, SMD_Packages:SOIC-14_N, F.Cu at (248.9, 84.3)
- C1: value 10µF -> 10nF; footprint Capacitors_SMD:CP_Elec_3x5.3 -> Capacitors_SMD:C_0402
- C2: footprint Capacitors_SMD:CP_Elec_3x5.3 -> Capacitors_SMD:CP_Elec_5x4.5
- C3: moved to B.Cu
- M1: footprint XBEE:XBEE -> XBEE:mDot
- SW1: footprint Buttons_Switches_SMD:SW_SPST_B3S-1000 -> Buttons_Switches_SMD:SW_SPST_EVQP7C
- U2: value NCS36000 -> IRA-E700; footprint SMD_Packages:SOIC-14_N -> PIR:IRA-E700
- moved C2 53.4 mm to (188.0, 96.5)
- moved SW1 32.4 mm to (203.2, 110.5), turned to 270 degrees
- moved M1 30.8 mm to (201.4, 116.6)
- moved U1 29.1 mm to (239.5, 117.3), turned to 180 degrees
- moved U2 27.0 mm to (213.6, 87.6)
- moved R1 25.1 mm to (235.2, 118.1)
- moved C1 19.0 mm to (248.2, 90.2), turned to 180 degrees
- moved R2 15.2 mm to (235.2, 117.1)
- moved C3 6.64 mm to (248.9, 84.6)
- moved C4 3.03 mm to (238.3, 120.7), turned to 180 degrees
Connections:
- C1 pad 1: +5V -> Net-(C1-Pad1)
- C1 pad 2: GND -> Net-(C1-Pad2)
- M1 pad 19: Net-(M1-Pad19) -> +3V3
- U1 pad 5: Net-(R3-Pad2) -> GND
Routing:
- net +3V3: track 0.00 -> 10.6 mm
- net GND: track 0.00 -> 10.5 mm, vias 0 -> 9
- net Net-(C8-Pad2): track 0.00 -> 6.60 mm
- net Net-(C1-Pad1): track 0.00 -> 4.53 mm
- net Net-(C1-Pad2): track 0.00 -> 4.16 mm
- net Net-(C6-Pad1): track 0.00 -> 4.13 mm
- net Net-(C8-Pad1): track 0.00 -> 3.58 mm
- net Net-(C10-Pad2): track 0.00 -> 2.64 mm
- net Net-(C7-Pad2): track 0.00 -> 2.56 mm
- net Net-(M1-Pad6): track 0.00 -> 1.82 mm
- net Net-(C5-Pad1): track 0.00 -> 1.75 mm
- net Net-(M1-Pad7): track 0.00 -> 1.67 mm
- net Net-(C9-Pad2): track 0.00 -> 1.59 mm
- added copper zone on B.Cu, net GND
- added copper zone on F.Cu, net GND

Commit message: test
Parts:
- added D1: LED, LEDs:LED_0805, F.Cu at (215.0, 64.5)
- added J1: Screw_Terminal_01x02, Connectors_Terminal_Blocks:TerminalBlock_Pheonix_MPT-2.54mm_2pol, F.Cu at (195.5, 93.0)
- added R3: 10k, Resistors_SMD:R_0805, B.Cu at (204.5, 78.5)
- C1, C10, C7, C8, C9: footprint Capacitors_SMD:C_0402 -> Capacitors_SMD:C_0805; moved to B.Cu
- C3: footprint Capacitors_SMD:C_0402 -> Capacitors_SMD:C_0805; moved to F.Cu
- C4: footprint Capacitors_SMD:C_0402 -> Capacitors_SMD:C_0805
- C5, C6, SW1, U3: moved to B.Cu
- M1: footprint XBEE:mDot -> STC:mDot
- R1, R2: footprint Resistors_SMD:R_0402 -> Resistors_SMD:R_0805
- R5, R6, R7, R8, R9: footprint Resistors_SMD:R_0402 -> Resistors_SMD:R_0805; moved to B.Cu
- RV1, RV2: footprint Potentiometers:Potentiometer_Trimmer-EVM3E -> STC:TRIM-EV1D-RMC
- U1: footprint BME280:BME280 -> STC:BME280
- U2: footprint PIR:IRA-E700 -> STC:IRA-E700
- moved C9 52.2 mm to (199.5, 90.5)
- moved R8 49.2 mm to (201.5, 90.5)
- moved R5 47.5 mm to (203.5, 94.0)
- moved C7 46.2 mm to (203.5, 90.5)
- moved SW1 44.8 mm to (194.6, 66.5), turned to 90 degrees
- moved C5 44.0 mm to (205.5, 94.0)
- moved U3 43.4 mm to (205.5, 83.5), turned to 180 degrees
- moved C1 41.7 mm to (206.5, 91.5), turned to 0 degrees
- moved R6 41.7 mm to (206.5, 89.5), turned to 0 degrees
- moved C6 40.2 mm to (207.5, 94.0)
- moved R9 39.4 mm to (207.5, 77.5)
- moved R2 37.4 mm to (207.5, 92.0)
- moved R7 37.1 mm to (209.5, 94.0)
- moved R1 36.7 mm to (207.5, 94.0)
- moved U1 36.6 mm to (212.7, 92.4)
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Connections:
- M1 pad 19: +3V3 -> Net-(M1-Pad19)
- M1 pad 20: Net-(M1-Pad20) -> +3V3
- U3 pad 12: Net-(U3-Pad12) -> Net-(M1-Pad15)
- U3 pad 8: Net-(U3-Pad8) -> Net-(M1-Pad19)
Routing:
- net Net-(C7-Pad2): track 2.56 -> 20.7 mm, vias 0 -> 1
- net Net-(C9-Pad2): track 1.59 -> 16.8 mm
- net +3V3: track 10.6 -> 3.49 mm
- net Net-(C1-Pad1): track 4.53 -> 0.00 mm
- net Net-(C1-Pad2): track 4.16 -> 0.00 mm
- net Net-(C6-Pad1): track 4.13 -> 0.00 mm
- net Net-(C8-Pad2): track 6.60 -> 3.30 mm
- net GND: track 10.5 -> 7.49 mm, vias 9 -> 0
- net Net-(C10-Pad2): track 2.64 -> 0.00 mm
- net Net-(C5-Pad1): track 1.75 -> 0.00 mm
- net Net-(M1-Pad7): track 1.67 -> 2.27 mm
- net Net-(C8-Pad1): track 3.58 -> 4.15 mm
- removed copper zone on F.Cu, net GND
Other:
- board outline added: 26 x 38 mm

Commit message: test
Parts:
- removed C2: 10µF, Capacitors_SMD:CP_Elec_5x4.5
- C1, C10, C7, C8, C9: footprint Capacitors_SMD:C_0805 -> Capacitors_SMD:C_0402
- C3, C4: footprint Capacitors_SMD:C_0805 -> Capacitors_SMD:C_0402; moved to B.Cu
- D1: footprint LEDs:LED_0805 -> LEDs:LED_0603
- R1, R2: footprint Resistors_SMD:R_0805 -> Resistors_SMD:R_0402; moved to B.Cu
- R3, R5, R6, R7, R8, R9: footprint Resistors_SMD:R_0805 -> Resistors_SMD:R_0402
- RV1, RV2: footprint STC:TRIM-EV1D-RMC -> Potentiometers:Potentiometer_Trimmer_Bourns_3296W
- SW1: footprint Buttons_Switches_SMD:SW_SPST_EVQP7C -> Buttons_Switches_THT:SW_PUSH_6mm_h5mm; moved to F.Cu
- U1: moved to B.Cu
- moved C4 32.2 mm to (199.0, 66.3)
- moved SW1 30.0 mm to (200.2, 96.0), turned to 180 degrees
- moved R1 28.4 mm to (193.4, 69.4), turned to 180 degrees
- moved C3 27.8 mm to (201.3, 69.5), turned to 270 degrees
- moved U1 26.1 mm to (200.2, 69.5)
- moved R2 25.7 mm to (195.2, 69.4)
- moved D1 19.3 mm to (213.4, 83.7), turned to 270 degrees
- moved J1 19.2 mm to (214.5, 95.7), turned to 90 degrees
- moved R5 14.3 mm to (198.2, 80.7), turned to 180 degrees
- moved C5 13.9 mm to (198.1, 82.3), turned to 0 degrees
- moved C6 13.6 mm to (198.1, 84.3), turned to 0 degrees
- moved R7 13.4 mm to (198.8, 86.0), turned to 180 degrees
- moved RV2 12.1 mm to (203.5, 95.0), turned to 180 degrees
- moved C9 11.0 mm to (201.2, 79.7), turned to 0 degrees
- moved C1 10.0 mm to (200.8, 83.3), turned to 270 degrees
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Connections:
- RV2 pad 1: Net-(R9-Pad2) -> +3V3
- RV2 pad 3: +3V3 -> Net-(R9-Pad2)
Routing:
- net +3V3: track 3.49 -> 104.5 mm
- net GND: track 7.49 -> 60.1 mm, vias 0 -> 26
- net Net-(M1-Pad5): track 0.00 -> 20.0 mm
- net Net-(M1-Pad7): track 2.27 -> 19.8 mm
- net Net-(M1-Pad6): track 2.29 -> 14.7 mm
- net Net-(R9-Pad2): track 0.00 -> 10.2 mm
- net Net-(C8-Pad2): track 3.30 -> 13.3 mm
- net Net-(M1-Pad19): track 0.00 -> 8.74 mm
- net Net-(C1-Pad2): track 0.00 -> 8.52 mm
- net Net-(C1-Pad1): track 0.00 -> 8.51 mm
- net Net-(C9-Pad2): track 16.8 -> 8.84 mm
- net Net-(M1-Pad15): track 0.00 -> 7.53 mm
- net Net-(C7-Pad2): track 20.7 -> 14.9 mm, vias 1 -> 0
- net Net-(D1-Pad1): track 0.00 -> 4.20 mm, vias 0 -> 1
- net Net-(C8-Pad1): track 4.15 -> 7.74 mm
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- added copper zone on F.Cu, net GND
