File: main.sch (KiCad schematic (older format))
At the start: 4 parts, among them M1 XBEE, U1 BME280, U2 NCS36000

Commit message: test
Parts:
- M1: footprint BME280:XBEE -> XBEE:XBEE-SMD
Changed lines of the file:
@@
 F 0 "M1" H 4300 4500 50  0000 L BNN
 F 1 "XBEE" H 5800 2800 50  0000 L BNN
-F 2 "BME280:XBEE" H 4400 2850 50  0001 C CNN
+F 2 "XBEE:XBEE-SMD" H 4400 2850 50  0001 C CNN
 F 3 "" H 5100 3750 60  0000 C CNN
 	1    5100 3750

Commit message: test
Parts:
- removed C1: CP, Capacitors_SMD:CP_Elec_3x5.3, symbol CP
- removed M1: XBEE, XBEE:XBEE-SMD, symbol XBEE
- removed U2: NCS36000, SMD_Packages:SOIC-14_N, symbol NCS36000
- added C2: 10µF, Capacitors_SMD:CP_Elec_3x5.3, symbol CP
- added C3, C4: 0.1µF, Capacitors_SMD:C_0402, symbol C_Small
- added C? (x2): 10nF, symbol C
- added C? (x2): 33µF, symbol C
- added C? (x3): 100nF, symbol C
- added M1: mDot, XBEE:XBEE, symbol mDot
- added R1, R2: 4.7k, Resistors_SMD:R_0402, symbol R
- added R3, R4: 0, Resistors_SMD:R_0402, symbol R
- added R? (x3): 10k, symbol R
- added R?: 43k, symbol R
- added R?: 51k, symbol R
- added RV? (x2): 1M, symbol POT
- added SW1: Reset, Buttons_Switches_SMD:SW_SPST_B3S-1000, symbol SW_Push
- added U?: NCS36000, symbol NCS36000
- added U?: IRA-E700, symbol IRA-E700
Connections:
- net labels removed: +5V
- wire segments 14 -> 114

Commit message: test
Parts:
- removed R3, R4: 0, Resistors_SMD:R_0402, symbol R
- C1, C10, C7, C8, C9: renamed from C?; footprint (none) -> Capacitors_SMD:C_0402
- C2: footprint Capacitors_SMD:CP_Elec_3x5.3 -> Capacitors_SMD:CP_Elec_5x4.5
- C5, C6: renamed from C?; footprint (none) -> Capacitors_SMD:C_0805
- M1: footprint XBEE:XBEE -> XBEE:mDot
- R5, R6, R7, R8, R9: renamed from R?; footprint (none) -> Resistors_SMD:R_0402
- RV1, RV2: renamed from RV?; footprint (none) -> Potentiometers:Potentiometer_Trimmer-EVM3E
- SW1: footprint Buttons_Switches_SMD:SW_SPST_B3S-1000 -> Buttons_Switches_SMD:SW_SPST_EVQP7C
- U2: renamed from U?; footprint (none) -> PIR:IRA-E700
- U3: renamed from U?; footprint (none) -> SMD_Packages:SOIC-14_N
Connections:
- net GND: now also U1.5 (SPI_SDO|I2C_ADR)

Commit message: test
Parts:
- added D1: LED, LEDs:LED_0805, symbol LED
- added J1: Screw_Terminal_01x02, Connectors_Terminal_Blocks:TerminalBlock_Pheonix_MPT-2.54mm_2pol, symbol Screw_Terminal_01x02
- added R3: 10k, Resistors_SMD:R_0805, symbol R
- C1, C10, C3, C4, C7, C8, C9: footprint Capacitors_SMD:C_0402 -> Capacitors_SMD:C_0805
- M1: footprint XBEE:mDot -> STC:mDot
- R1, R2, R5, R6, R7, R8, R9: footprint Resistors_SMD:R_0402 -> Resistors_SMD:R_0805
- RV1, RV2: footprint Potentiometers:Potentiometer_Trimmer-EVM3E -> STC:TRIM-EV1D-RMC
- U1: footprint BME280:BME280 -> STC:BME280
- U2: footprint PIR:IRA-E700 -> STC:IRA-E700
Connections:
- net +3V3: now also M1.20 (BP1|ADC|PWM1/3|5V), J1.1 (Pin_1); no longer M1.19 (PB0|ADC|PWM1/2)
- net GND: now also D1.2 (A), J1.2 (Pin_2)
- net at M1.15 (PC1|ASSOCIATE|ADC|5V): now also U3.12 (MODE)
- net at U3.8 (OUT): now also M1.19 (PB0|ADC|PWM1/2)
- net at U3.9 (LED): now also R3.2
- new net: D1.1 (K), R3.1
Other:
- moved on the sheet: C1, C10, C5, C6, C7, C8, C9, M1, R5, R6, R7, R8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

Commit message: test
Parts:
- C1, C10, C3, C4, C7, C8, C9: footprint Capacitors_SMD:C_0805 -> Capacitors_SMD:C_0402
- D1: footprint LEDs:LED_0805 -> LEDs:LED_0603
- R1, R2, R3, R5, R6, R7, R8, R9: footprint Resistors_SMD:R_0805 -> Resistors_SMD:R_0402
- RV1, RV2: footprint STC:TRIM-EV1D-RMC -> Potentiometers:Potentiometer_Trimmer_Bourns_3296W
- SW1: footprint Buttons_Switches_SMD:SW_SPST_EVQP7C -> Buttons_Switches_THT:SW_PUSH_6mm_h5mm
Connections:
- net +3V3: now also RV2.1; no longer RV2.3
- net at R9.2: now also RV2.3; no longer RV2.1
Changed lines of the file:
@@
 F 0 "R1" V 4380 1400 50  0000 C CNN
 F 1 "4.7k" V 4300 1400 50  0000 C CNN
-F 2 "Resistors_SMD:R_0805" V 4230 1400 50  0001 C CNN
+F 2 "Resistors_SMD:R_0402" V 4230 1400 50  0001 C CNN
 F 3 "" H 4300 1400 50  0001 C CNN
 	1    4300 1400
@@
 F 0 "R2" V 4580 1400 50  0000 C CNN
 F 1 "4.7k" V 4500 1400 50  0000 C CNN
-F 2 "Resistors_SMD:R_0805" V 4430 1400 50  0001 C CNN
+F 2 "Resistors_SMD:R_0402" V 4430 1400 50  0001 C CNN
 F 3 "" H 4500 1400 50  0001 C CNN
 	1    4500 1400
@@
 F 0 "C4" H 2310 1970 50  0000 L CNN
 F 1 "0.1µF" H 2310 1820 50  0000 L CNN
-F 2 "Capacitors_SMD:C_0805" H 2300 1900 50  0001 C CNN
+F 2 "Capacitors_SMD:C_0402" H 2300 1900 50  0001 C CNN
 F 3 "" H 2300 1900 50  0001 C CNN
 	1    2300 1900
@@
 F 0 "C3" H 1960 1970 50  0000 L CNN
 F 1 "0.1µF" H 1960 1820 50  0000 L CNN
-F 2 "Capacitors_SMD:C_0805" H 1950 1900 50  0001 C CNN
+F 2 "Capacitors_SMD:C_0402" H 1950 1900 50  0001 C CNN
 F 3 "" H 1950 1900 50  0001 C CNN
 	1    1950 1900
@@
 F 0 "SW1" H 4700 3050 50  0000 L CNN
 F 1 "Reset" H 4650 2890 50  0000 C CNN
-F 2 "Buttons_Switches_SMD:SW_SPST_EVQP7C" H 4650 3150 50  0001 C CNN
+F 2 "Buttons_Switches_THT:SW_PUSH_6mm_h5mm" H 4650 3150 50  0001 C CNN
 F 3 "" H 4650 3150 50  0001 C CNN
 	1    4650 2950
@@
 F 0 "C8" V 2450 4900 50  0000 L CNN
 F 1 "10nF" V 2450 4600 50  0000 L CNN
-F 2 "Capacitors_SMD:C_0805" H 2538 4700 50  0001 C CNN
+F 2 "Capacitors_SMD:C_0402" H 2538 4700 50  0001 C CNN
 F 3 "" H 2500 4850 50  0001 C CNN
 	1    2500 4850
@@
 F 0 "R7" V 1750 4850 50  0000 C CNN
 F 1 "10k" V 1850 4850 50  0000 C CNN
-F 2 "Resistors_SMD:R_0805" V 1780 4850 50  0001 C CNN
+F 2 "Resistors_SMD:R_0402" V 1780 4850 50  0001 C CNN
 F 3 "" H 1850 4850 50  0001 C CNN
 	1    1850 4850
@@
 F 0 "C1" V 950 5600 50  0000 L CNN
 F 1 "10nF" V 950 5300 50  0000 L CNN
-F 2 "Capacitors_SMD:C_0805" H 938 5400 50  0001 C CNN
+F 2 "Capacitors_SMD:C_0402" H 938 5400 50  0001 C CNN
 F 3 "" H 900 5550 50  0001 C CNN
 	1    900  5550
@@
 F 0 "R6" V 1000 5550 50  0000 C CNN
 F 1 "10k" V 1100 5550 50  0000 C CNN
-F 2 "Resistors_SMD:R_0805" V 1030 5550 50  0001 C CNN
+F 2 "Resistors_SMD:R_0402" V 1030 5550 50  0001 C CNN
 F 3 "" H 1100 5550 50  0001 C CNN
 	1    1100 5550
@@
 F 0 "R5" V 980 6350 50  0000 C CNN
 F 1 "10k" V 900 6350 50  0000 C CNN
-F 2 "Resistors_SMD:R_0805" V 830 6350 50  0001 C CNN
+F 2 "Resistors_SMD:R_0402" V 830 6350 50  0001 C CNN
 F 3 "" H 900 6350 50  0001 C CNN
 	1    900  6350
@@
 F 0 "C9" V 2600 6400 50  0000 L CNN
 F 1 "100nF" V 2600 6050 50  0000 L CNN
-F 2 "Capacitors_SMD:C_0805" H 2688 6200 50  0001 C CNN
+F 2 "Capacitors_SMD:C_0402" H 2688 6200 50  0001 C CNN
 F 3 "" H 2650 6350 50  0001 C CNN
 	1    2650 6350
@@
 F 0 "R8" V 2280 6350 50  0000 C CNN
 F 1 "43k" V 2200 6350 50  0000 C CNN
-F 2 "Resistors_SMD:R_0805" V 2130 6350 50  0001 C CNN
+F 2 "Resistors_SMD:R_0402" V 2130 6350 50  0001 C CNN
 F 3 "" H 2200 6350 50  0001 C CNN
 	1    2200 6350
@@
 F 0 "C7" V 2400 6400 50  0000 L CNN
 F 1 "100nF" V 2400 6050 50  0000 L CNN
-F 2 "Capacitors_SMD:C_0805" H 2488 6200 50  0001 C CNN
+F 2 "Capacitors_SMD:C_0402" H 2488 6200 50  0001 C CNN
 F 3 "" H 2450 6350 50  0001 C CNN
 	1    2450 6350
@@
 F 0 "C10" H 4725 5600 50  0000 L CNN
 F 1 "100nF" H 4725 5400 50  0000 L CNN
-F 2 "Capacitors_SMD:C_0805" H 4738 5350 50  0001 C CNN
+F 2 "Capacitors_SMD:C_0402" H 4738 5350 50  0001 C CNN
 F 3 "" H 4700 5500 50  0001 C CNN
 	1    4700 5500
@@
 F 0 "R9" V 4780 5050 50  0000 C CNN
 F 1 "51k" V 4700 5050 50  0000 C CNN
-F 2 "Resistors_SMD:R_0805" V 4630 5050 50  0001 C CNN
+F 2 "Resistors_SMD:R_0402" V 4630 5050 50  0001 C CNN
 F 3 "" H 4700 5050 50  0001 C CNN
 	1    4700 5050
@@
 F 0 "RV2" V 4600 4700 50  0000 C CNN
 F 1 "1M" V 4700 4700 50  0000 C CNN
-F 2 "STC:TRIM-EV1D-RMC" H 4700 4700 50  0001 C CNN
+F 2 "Potentiometers:Potentiometer_Trimmer_Bourns_3296W" H 4700 4700 50  0001 C CNN
 F 3 "" H 4700 4700 50  0001 C CNN
 	1    4700 4700
-	-1   0    0    1
+	-1   0    0    -1
 $EndComp
 Wire Wire Line
@@
 F 0 "RV1" V 2600 5050 50  0000 C CNN
 F 1 "1M" V 2500 5150 50  0000 C CNN
-F 2 "STC:TRIM-EV1D-RMC" H 2500 5150 50  0001 C CNN
+F 2 "Potentiometers:Potentiometer_Trimmer_Bourns_3296W" H 2500 5150 50  0001 C CNN
 F 3 "" H 2500 5150 50  0001 C CNN
 	1    2500 5150
@@
 F 0 "D1" H 4350 6400 50  0000 C CNN
 F 1 "LED" H 4350 6200 50  0000 C CNN
-F 2 "LEDs:LED_0805" H 4350 6300 50  0001 C CNN
+F 2 "LEDs:LED_0603" H 4350 6300 50  0001 C CNN
 F 3 "" H 4350 6300 50  0001 C CNN
 	1    4350 6300
@@
 F 0 "R3" V 4250 5950 50  0000 C CNN
 F 1 "10k" V 4350 5950 50  0000 C CNN
-F 2 "Resistors_SMD:R_0805" V 4280 5950 50  0001 C CNN
+F 2 "Resistors_SMD:R_0402" V 4280 5950 50  0001 C CNN
 F 3 "" H 4350 5950 50  0001 C CNN
 	1    4350 5950
