File: type2/main.kicad_pcb (KiCad board)
At the start: 2 copper layers, 35 x 38 mm, 17 parts, among them J1 Conn_01x02, M1 mDot, SW1 SW_Push, U1 AMN31111, U2 BME280, U3 MIC5219-3.3

Commit message: test
Parts:
- moved R1 0.35 mm to (158.4, 80.7)
- moved R2 0.20 mm to (158.4, 82.7)
