File: type2/main.kicad_pcb (KiCad board)
At the start: 2 copper layers, 35 x 38 mm, 17 parts, among them J1 Conn_01x02, M1 mDot, SW1 SW_Push, U1 AMN31111, U2 BME280, U3 MIC5219-3.3

Commit message: Improved design
Parts:
- C3, C4, C5: footprint Capacitors_SMD:C_0402 -> Capacitors_SMD:C_0603
- PIR Sensor: renamed from U1; footprint STC:AMN31111 -> AMN31111
- R1, R2: footprint Resistors_SMD:R_0402 -> Resistors_SMD:R_0603
- moved R1 1.39 mm to (159.8, 80.7)
- moved R2 1.36 mm to (159.8, 82.7)
- moved C5 1.30 mm to (152.5, 84.7), turned to 180 degrees
- moved PIR Sensor 1.12 mm to (167.5, 85.0), turned to 90 degrees
- moved C4 0.20 mm to (152.5, 80.0)
Connections:
- M1 pad 11: Net-(M1-Pad11) -> (no net)
- M1 pad 12: Net-(M1-Pad12) -> (no net)
- M1 pad 13: Net-(M1-Pad13) -> (no net)
- M1 pad 14: Net-(M1-Pad14) -> (no net)
- M1 pad 15: Net-(M1-Pad15) -> (no net)
- M1 pad 16: Net-(M1-Pad16) -> (no net)
- M1 pad 17: Net-(M1-Pad17) -> (no net)
- M1 pad 18: Net-(M1-Pad18) -> (no net)
- M1 pad 19: Net-(M1-Pad19) -> (no net)
- M1 pad 2: Net-(M1-Pad2) -> (no net)
- M1 pad 20: Net-(M1-Pad20) -> (no net)
- M1 pad 24: Net-(M1-Pad24) -> (no net)
- M1 pad 26: Net-(M1-Pad26) -> (no net)
- M1 pad 27: Net-(M1-Pad27) -> (no net)
- M1 pad 28: Net-(M1-Pad28) -> (no net)
- M1 pad 29: Net-(M1-Pad29) -> (no net)
- M1 pad 3: Net-(M1-Pad3) -> (no net)
- M1 pad 30: Net-(M1-Pad30) -> (no net)
- M1 pad 31: Net-(M1-Pad31) -> (no net)
- M1 pad 4: Net-(M1-Pad4) -> (no net)
- M1 pad 8: Net-(M1-Pad8) -> (no net)
- U3 pad 4: Net-(U3-Pad4) -> (no net)
Routing:
- net +3V3: track 58.1 -> 46.9 mm
- net -BATT: track 7.05 -> 14.3 mm
- net Net-(M1-Pad5): track 22.5 -> 18.6 mm
- net PIR_Out: track 11.6 -> 9.25 mm
- net SDA: track 4.00 -> 4.98 mm
- net SCL: track 4.07 -> 4.98 mm
Other:
- board text added: "Hole 30 x 33 mm Edge 35 x 38 mm"
- board text added: "P1 3.3V"
- board text added: "P10 GND"
- board text added: "P11"
- board text added: "P12"
- board text added: "P13"
- board text added: "P14"
- board text added: "P15"
- board text added: "P16"
- board text added: "P17"
- board text added: "P18"
- board text added: "P19"
- board text added: "P2"
- board text added: "P20"
- board text added: "P24"
- board text added: "P25 GND"
- board text added: "P26"
- board text added: "P27"
- board text added: "P28"
- board text added: "P29"
- board text added: "P3"
- board text added: "P30"
- board text added: "P31"
- board text added: "P4"
- board text added: "P5 NRESET"
- board text added: "P6 SCL"
- board text added: "P7 SDA"
- board text added: "P8"
- board text added: "P9 PIR"
- board text added: "Power in 3.3V..12V JST_PH"
- board text added: "VREG"
- board text removed: "3.3V-12V"
- board text removed: "NRESET P5"
- board text removed: "PIR_Out PA11 P9"
- board text removed: "Power in"
