File: type2/main.sch (KiCad schematic (older format))
At the start: 13 parts, among them J1 Conn_01x02, M1 mDot, SW1 SW_Push, U1 AMN31111, U2 BME280, U3 MIC5219-3.3

Commit message: test
Parts:
- added R?: R, Resistors_SMD:R_0402, symbol R
Connections:
- net +3V3: now also R?.1
- net PIR_Out: now also R?.2
Changed lines of the file:
@@
 LIBS:PIR_Panasonic
 LIBS:Bosch_Sensortec
+LIBS:main-cache
 EELAYER 25 0
 EELAYER END
@@
 Wire Wire Line
 	8600 4400 8350 4400
+$Comp
+L R R?
+U 1 1 59C95279
+P 3600 1800
+F 0 "R?" V 3680 1800 50  0000 C CNN
+F 1 "R" V 3600 1800 50  0000 C CNN
+F 2 "Resistors_SMD:R_0402" V 3530 1800 50  0001 C CNN
+F 3 "" H 3600 1800 50  0001 C CNN
+	1    3600 1800
+	1    0    0    -1
+$EndComp
+Wire Wire Line
+	3600 1950 3600 2050
+Connection ~ 3600 2050
+$Comp
+L +3.3V #PWR?
+U 1 1 59C95564
+P 3600 1600
+F 0 "#PWR?" H 3600 1450 50  0001 C CNN
+F 1 "+3.3V" H 3600 1740 50  0000 C CNN
+F 2 "" H 3600 1600 50  0001 C CNN
+F 3 "" H 3600 1600 50  0001 C CNN
+	1    3600 1600
+	1    0    0    -1
+$EndComp
+Wire Wire Line
+	3600 1600 3600 1650
 $EndSCHEMATC
