File: type2/main.sch (KiCad schematic (older format))
At the start: 13 parts, among them J1 Conn_01x02, M1 mDot, SW1 SW_Push, U1 AMN31111, U2 BME280, U3 MIC5219-3.3

Commit message: Improved design
Parts:
- C3, C4, C5: footprint Capacitors_SMD:C_0402 -> Capacitors_SMD:C_0603
- R1, R2: footprint Resistors_SMD:R_0402 -> Resistors_SMD:R_0603
Changed lines of the file:
@@
 LIBS:PIR_Panasonic
 LIBS:Bosch_Sensortec
+LIBS:main-cache
 EELAYER 25 0
 EELAYER END
@@
 F 0 "R1" V 7680 1450 50  0000 C CNN
 F 1 "R" V 7600 1450 50  0000 C CNN
-F 2 "Resistors_SMD:R_0402" V 7530 1450 50  0001 C CNN
+F 2 "Resistors_SMD:R_0603" V 7530 1450 50  0001 C CNN
 F 3 "" H 7600 1450 50  0001 C CNN
 	1    7600 1450
@@
 F 0 "R2" V 7880 1450 50  0000 C CNN
 F 1 "R" V 7800 1450 50  0000 C CNN
-F 2 "Resistors_SMD:R_0402" V 7730 1450 50  0001 C CNN
+F 2 "Resistors_SMD:R_0603" V 7730 1450 50  0001 C CNN
 F 3 "" H 7800 1450 50  0001 C CNN
 	1    7800 1450
@@
 F 0 "C5" H 5575 1950 50  0000 L CNN
 F 1 "100nF" H 5575 1750 50  0000 L CNN
-F 2 "Capacitors_SMD:C_0402" H 5588 1700 50  0001 C CNN
+F 2 "Capacitors_SMD:C_0603" H 5588 1700 50  0001 C CNN
 F 3 "" H 5550 1850 50  0001 C CNN
 	1    5550 1850
@@
 F 0 "C3" H 3325 5350 50  0000 L CNN
 F 1 "100nF" H 3325 5150 50  0000 L CNN
-F 2 "Capacitors_SMD:C_0402" H 3338 5100 50  0001 C CNN
+F 2 "Capacitors_SMD:C_0603" H 3338 5100 50  0001 C CNN
 F 3 "" H 3300 5250 50  0001 C CNN
 	1    3300 5250
@@
 F 0 "C4" H 5225 1950 50  0000 L CNN
 F 1 "100nF" H 5225 1750 50  0000 L CNN
-F 2 "Capacitors_SMD:C_0402" H 5238 1700 50  0001 C CNN
+F 2 "Capacitors_SMD:C_0603" H 5238 1700 50  0001 C CNN
 F 3 "" H 5200 1850 50  0001 C CNN
 	1    5200 1850
